File: pcbs/common/left.kicad_sch (KiCad schematic)
At the start: 88 parts

Commit message: Schematic rearangement
Parts:
- removed C? (x2): 27p, Capacitor_SMD:C_0402_1005Metric, symbol Device:C_Small
- removed C? (x2): 10u, Capacitor_SMD:C_0402_1005Metric, symbol Device:C_Small
- removed EXLED? (x2), LED? (x21): YS-SK6812MINI-E, kbd_local:YS-SK6812MINI-E, symbol kbd_local:YS-SK6812MINI-E
- removed F?: BSMD0603-050-12V, Fuse:Fuse_0603_1608Metric, symbol Device:Fuse
- removed R?: 1k, Resistor_SMD:R_0402_1005Metric, symbol Device:R
- removed U?: NCP1117LPST33T3G, Package_TO_SOT_SMD:SOT-223-3_TabPin2, symbol Regulator_Linear:NCP1117-3.3_SOT223
- removed Y?: 12MHz 18pF, Crystal:Crystal_SMD_3225-4Pin_3.2x2.5mm, symbol Device:Crystal_GND24_Small
- removed ZD?: ESD5Z5V0C, Diode_SMD:D_SOD-523, symbol Diode:ESD5Zxx
- added C1, C2: 27p, Capacitor_SMD:C_0402_1005Metric, symbol Device:C_Small
- added C11, C6: 10u, Capacitor_SMD:C_0402_1005Metric, symbol Device:C_Small
- added EXLED1, EXLED2, LED1, LED10, LED11, LED12, LED13, LED14, LED15, LED16, LED17, LED18, LED19, LED2, LED20, LED21, LED3, LED4, LED5, LED6, LED7, LED8, LED9: YS-SK6812MINI-E, kbd_local:YS-SK6812MINI-E, symbol kbd_local:YS-SK6812MINI-E
- added F1: BSMD0603-050-12V, Fuse:Fuse_0603_1608Metric, symbol Device:Fuse
- added R3: 1k, Resistor_SMD:R_0402_1005Metric, symbol Device:R
- added U2: NCP1117LPST33T3G, Package_TO_SOT_SMD:SOT-223-3_TabPin2, symbol Regulator_Linear:NCP1117-3.3_SOT223
- added Y1: 12MHz 18pF, Crystal:Crystal_SMD_3225-4Pin_3.2x2.5mm, symbol Device:Crystal_GND24_Small
- added ZD1: ESD5Z5V0C, Diode_SMD:D_SOD-523, symbol Diode:ESD5Zxx
Connections:
- net KEYEX2 is gone; now on net GND: EXSW?.S2, U?.11 (GPIO8)
- net +3V3: now also C11.1, U2.2 (VO)
- net +5V: now also C6.1, F1.2, U2.3 (VI)
- net GND: now also EXSW?.B, C1.1, C11.2, C2.1, C6.2, EXLED1.3 (VSS), EXLED2.3 (VSS), LED1.3 (VSS), LED10.3 (VSS), LED11.3 (VSS), LED12.3 (VSS), LED13.3 (VSS), LED14.3 (VSS), LED15.3 (VSS), LED16.3 (VSS), LED17.3 (VSS), LED18.3 (VSS), LED19.3 (VSS), LED2.3 (VSS), LED20.3 (VSS), LED21.3 (VSS), LED3.3 (VSS), LED4.3 (VSS), LED5.3 (VSS), LED6.3 (VSS), LED7.3 (VSS), LED8.3 (VSS), LED9.3 (VSS), U2.1 (GND), Y1.2, Y1.4, ZD1.2 (A); no longer EXSW?.C, EXSW?.S1
- net KEYEX1: now also EXSW?.A; no longer EXSW?.S2
- net RE0A: now also EXSW?.S2; no longer EXSW?.A
- net REB: now also EXSW?.S1; no longer EXSW?.B
- net VBUS: now also F1.1, ZD1.1 (K)
- net at D?.1 (K): now also JP1.2 (B)
- net XIN: now reaches U?.20 (XIN)
- net XIN: now also C1.2, Y1.1
- net XOUT: now reaches U?.21 (XOUT)
- net XOUT: now also R3.2
- net LED_+5V: now reaches JP1.1 (A)
- net LED_+5V: now also EXLED1.1 (VDD), EXLED2.1 (VDD), LED1.1 (VDD), LED10.1 (VDD), LED11.1 (VDD), LED12.1 (VDD), LED13.1 (VDD), LED14.1 (VDD), LED15.1 (VDD), LED16.1 (VDD), LED17.1 (VDD), LED18.1 (VDD), LED19.1 (VDD), LED2.1 (VDD), LED20.1 (VDD), LED21.1 (VDD), LED3.1 (VDD), LED4.1 (VDD), LED5.1 (VDD), LED6.1 (VDD), LED7.1 (VDD), LED8.1 (VDD), LED9.1 (VDD)
- new net: C2.2, R3.1, Y1.3
- no-connect marks 3 -> 2
Other:
- note added: "Crystal"
- note added: "Voltage Regulation"
- moved on the sheet: C?, D?, EXSW?, J?, JP1, R?, SMDSW?, SW?, U?
